File: boards/addons/02_7seg_led_direct/02_7seg_led_direct.kicad_sch (KiCad schematic)
At the start: 12 parts, among them J1 Conn_01x08_Socket, J2 Conn_01x04_Socket, U1 74AHC541

Commit message: かいろず
Parts:
- added U2: ~, OptoSupply:OSL10561, symbol OptoSupply:OSL10561
Connections:
- net GND: now also U2.3 (Common), U2.8 (Common)
- net LED_A: now also U2.7 (A)
- net LED_B: now also U2.6 (B)
- net LED_C: now also U2.4 (C)
- net LED_D: now also U2.2 (D)
- net LED_DP: now also U2.5 (DP)
- net LED_E: now also U2.1 (E)
- net LED_F: now also U2.9 (F)
- net LED_G: now also U2.10 (G)
