File: boards/addons/02_7seg_led_direct/02_7seg_led_direct.kicad_pcb (KiCad board)
At the start: 2 copper layers, 47.5 x 72 mm, 13 parts, among them J1 Conn_01x08_Socket, J2 Conn_01x04_Socket, U1 74AHC541

Commit message: シルクの追加とベタのテコ入れ
Other:
- board text added: "74HC541"
Changed lines of the file:
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@@
 			(pinfunction "GND")
 			(pintype "power_in")
+			(thermal_bridge_angle 45)
 		)
 		(pad "11" thru_hole oval
@@
 		)
 		(fp_text user "${REFERENCE}"
-			(at 0 8.89 360)
+			(at 0 8.89 0)
 			(layer "F.Fab")
 			(effects
@@
 			)
 			(justify right)
+		)
+	)
+	(gr_text "74HC541"
+		(at 114.3 119.38 -90)
+		(layer "F.SilkS")
+		(effects
+			(font
+				(size 1 1)
+				(thickness 0.1)
+			)
 		)
 	)
@@
 	)
 	(zone
-		(net 2)
-		(net_name "+3.3V")
-		(layer "F.Cu")
-		(hatch edge 0.5)
-		(priority 1)
-		(connect_pads
-			(clearance 0.5)
-		)
-		(min_thickness 0.25)
-		(filled_areas_thickness no)
-		(fill yes
-			(thermal_gap 0.5)
-			(thermal_bridge_width 0.5)
-		)
-		(polygon
-			(pts
-				(xy 104.775 94.996) (xy 106.934 94.996) (xy 106.934 98.044) (xy 105.41 98.044) (xy 105.156 98.298)
-				(xy 105.156 104.902) (xy 106.934 106.68) (xy 106.934 108.204) (xy 105.029 108.204) (xy 103.759 106.934)
-				(xy 103.759 96.012)
-			)
-		)
-	)
-	(zone
 		(net 0)
 		(net_name "")
-		(layer "B.Cu")
+		(layer "F.Cu")
 		(hatch edge 0.5)
 		(connect_pads
@@
 		(polygon
 			(pts
-				(xy 137.16 113.157) (xy 137.16 130.937) (xy 139.7 130.937) (xy 139.7 113.157)
+				(xy 105.41 97.536) (xy 106.426 97.536) (xy 106.426 95.504) (xy 105.41 95.504)
+			)
+		)
+	)
+	(zone
+		(net 2)
+		(net_name "+3.3V")
+		(layer "F.Cu")
+		(hatch edge 0.5)
+		(priority 1)
+		(connect_pads
+			(clearance 0.5)
+		)
+		(min_thickness 0.25)
+		(filled_areas_thickness no)
+		(fill yes
+			(thermal_gap 0.5)
+			(thermal_bridge_width 0.5)
+		)
+		(polygon
+			(pts
+				(xy 104.775 94.996) (xy 106.934 94.996) (xy 106.934 98.044) (xy 105.41 98.044) (xy 105.156 98.298)
+				(xy 105.156 104.902) (xy 106.934 106.68) (xy 106.934 108.204) (xy 105.029 108.204) (xy 103.759 106.934)
+				(xy 103.759 96.012)
 			)
 		)
@@
 		(polygon
 			(pts
-				(xy 142.24 88.9) (xy 144.78 88.9) (xy 144.78 86.36) (xy 142.24 86.36)
+				(xy 137.16 113.157) (xy 137.16 130.937) (xy 139.7 130.937) (xy 139.7 113.157)
 			)
 		)
@@
 		(polygon
 			(pts
-				(xy 116.84 107.95) (xy 116.84 110.236) (xy 119.38 110.236) (xy 119.38 107.95)
+				(xy 106.934 100.584) (xy 107.95 100.584) (xy 107.95 102.616) (xy 106.934 102.616)
 			)
 		)
@@
 		(polygon
 			(pts
-				(xy 142.24 104.14) (xy 144.78 104.14) (xy 144.78 101.6) (xy 142.24 101.6)
+				(xy 142.24 88.9) (xy 144.78 88.9) (xy 144.78 86.36) (xy 142.24 86.36)
 			)
 		)
@@
 		(polygon
 			(pts
-				(xy 105.41 93.98) (xy 105.41 100.076) (xy 107.95 100.076) (xy 107.95 93.98)
+				(xy 116.84 107.95) (xy 116.84 110.236) (xy 119.38 110.236) (xy 119.38 107.95)
 			)
 		)
@@
 		(polygon
 			(pts
-				(xy 134.62 88.9) (xy 137.16 88.9) (xy 137.16 86.36) (xy 134.62 86.36)
+				(xy 105.41 100.584) (xy 106.426 100.584) (xy 106.426 102.616) (xy 105.41 102.616)
 			)
 		)
@@
 		(polygon
 			(pts
-				(xy 134.62 104.14) (xy 137.16 104.14) (xy 137.16 101.6) (xy 134.62 101.6)
+				(xy 142.24 104.14) (xy 144.78 104.14) (xy 144.78 101.6) (xy 142.24 101.6)
 			)
 		)
@@
 		(polygon
 			(pts
-				(xy 116.84 110.744) (xy 116.84 130.683) (xy 119.38 130.683) (xy 119.38 110.744)
+				(xy 105.41 93.98) (xy 105.41 100.076) (xy 107.95 100.076) (xy 107.95 93.98)
 			)
 		)
@@
 		(polygon
 			(pts
-				(xy 110.49 69.85) (xy 110.49 72.39) (xy 130.81 72.39) (xy 130.81 69.85)
+				(xy 134.62 88.9) (xy 137.16 88.9) (xy 137.16 86.36) (xy 134.62 86.36)
 			)
 		)
@@
 		(polygon
 			(pts
-				(xy 109.22 108.204) (xy 109.22 130.556) (xy 111.76 130.556) (xy 111.76 108.204)
-			)
-		)
+				(xy 134.62 104.14) (xy 137.16 104.14) (xy 137.16 101.6) (xy 134.62 101.6)
+			)
+		)
+	)
+	(zone
+		(net 0)
+		(net_name "")
+		(layer "B.Cu")
+		(hatch edge 0.5)
+		(connect_pads
+			(clearance 0)
+		)
+		(min_thickness 0.25)
+		(filled_areas_thickness no)
+		(keepout
+			(tracks allowed)
+			(vias allowed)
+			(pads allowed)
+			(copperpour not_allowed)
+			(footprints allowed)
+		)
+		(fill
+			(thermal_gap 0.5)
+			(thermal_bridge_width 0.5)
+		)
+		(polygon
+			(pts
+				(xy 116.84 110.744) (xy 116.84 130.683) (xy 119.38 130.683) (xy 119.38 110.744)
+			)
+		)
+	)
+	(zone
+		(net 0)
+		(net_name "")
+		(layer "B.Cu")
+		(hatch edge 0.5)
+		(connect_pads
+			(clearance 0)
+		)
+		(min_thickness 0.25)
+		(filled_areas_thickness no)
+		(keepout
+			(tracks allowed)
+			(vias allowed)
+			(pads allowed)
+			(copperpour not_allowed)
+			(footprints allowed)
+		)
+		(fill
+			(thermal_gap 0.5)
+			(thermal_bridge_width 0.5)
+		)
+		(polygon
+			(pts
+				(xy 110.49 69.85) (xy 110.49 72.39) (xy 130.81 72.39) (xy 130.81 69.85)
+			)
+		)
+	)
+	(zone
+		(net 0)
+		(net_name "")
+		(layer "B.Cu")
+		(hatch edge 0.5)
+		(connect_pads
+			(clearance 0)
+		)
+		(min_thickness 0.25)
+		(filled_areas_thickness no)
+		(keepout
+			(tracks allowed)
+			(vias allowed)
+			(pads allowed)
+			(copperpour not_allowed)
+			(footprints allowed)
+		)
+		(fill
+			(thermal_gap 0.5)
+			(thermal_bridge_width 0.5)
+		)
+		(polygon
+			(pts
+				(xy 109.22 108.204) (xy 109.22 129.032) (xy 110.49 130.302) (xy 111.76 129.032) (xy 111.76 108.204)
+			)
+		)

Commit message: 改番
Other:
- board text added: "7 segments LED with Direct Drive v0.2"
- board text removed: "7 segments LED with Direct Drive v0.1"
Changed lines of the file:
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@@
 		)
 	)
-	(gr_text "7 segments LED with Direct Drive v0.1"
+	(gr_text "7 segments LED with Direct Drive v0.2"
 		(at 110.49 134.62 0)
 		(layer "F.SilkS")
