File: boards/addons/01_sw_and_led/01_sw_and_led.kicad_pcb (KiCad board)
At the start: 2 copper layers, 47.5 x 72 mm, 8 parts, among them J1 Conn_01x04_Socket, J2 Conn_01x04_Socket, SW1 SW_Push, SW2 SW_Push

Commit message: ナンバリング修正
Parts:
- removed R3, R4: R, Resistor_THT:R_Axial_DIN0207_L6.3mm_D2.5mm_P10.16mm_Horizontal
- added R1: R, Resistor_THT:R_Axial_DIN0207_L6.3mm_D2.5mm_P10.16mm_Horizontal, F.Cu at (153.7, 80.8)
- added R2: R, Resistor_THT:R_Axial_DIN0207_L6.3mm_D2.5mm_P10.16mm_Horizontal, F.Cu at (166.4, 80.8)

Commit message: 改番
Other:
- board text added: "SW and LED board for Digital IO v0.2"
- board text removed: "SW and LED board for Digital IO v0.1"
Changed lines of the file:
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@@
 		)
 	)
-	(gr_text "SW and LED board for Digital IO v0.1"
+	(gr_text "SW and LED board for Digital IO v0.2"
 		(at 135.89 134.62 0)
 		(layer "F.SilkS")
