File: boards/addons/03_7seg_led_595/03_7seg_led_595.kicad_pcb (KiCad board)
At the start: 2 copper layers, 47.5 x 72 mm, 16 parts, among them J1 Conn_01x05_Socket, J2 Conn_01x04_Socket, U1 74HC595

Commit message: シルクの追加とベタのテコ入れ その 2
Other:
- board text added: "74HC595"
Changed lines of the file:
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@@
 		)
 		(fp_text user "${REFERENCE}"
-			(at 0 5.08 360)
+			(at 0 5.08 0)
 			(layer "F.Fab")
 			(effects
@@
 		)
 	)
+	(gr_text "74HC595"
+		(at 142.24 132.08 0)
+		(layer "F.SilkS")
+		(effects
+			(font
+				(size 1 1)
+				(thickness 0.1)
+			)
+		)
+	)
 	(gr_text "ENABLE"
 		(at 137.16 78.74 90)
@@
 			)
 		)
+	)
+	(zone
+		(net 0)
+		(net_name "")
+		(layer "B.Cu")
+		(hatch edge 0.5)
+		(connect_pads
+			(clearance 0)
+		)
+		(min_thickness 0.25)
+		(filled_areas_thickness no)
+		(keepout
+			(tracks allowed)
+			(vias allowed)
+			(pads allowed)
+			(copperpour not_allowed)
+			(footprints allowed)
+		)
+		(fill
+			(thermal_gap 0.5)
+			(thermal_bridge_width 0.5)
+		)
+		(polygon
+			(pts
+				(xy 120.65 105.664) (xy 121.666 105.664) (xy 121.666 107.696) (xy 120.65 107.696)
+			)
+		)
+	)
+	(zone
+		(net 0)
+		(net_name "")
+		(layer "B.Cu")
+		(hatch edge 0.5)
+		(connect_pads
+			(clearance 0)
+		)
+		(min_thickness 0.25)
+		(filled_areas_thickness no)
+		(keepout
+			(tracks allowed)
+			(vias allowed)
+			(pads allowed)
+			(copperpour not_allowed)
+			(footprints allowed)
+		)
+		(fill
+			(thermal_gap 0.5)
+			(thermal_bridge_width 0.5)
+		)
+		(polygon
+			(pts
+				(xy 122.174 105.664) (xy 123.19 105.664) (xy 123.19 107.696) (xy 122.174 107.696)
+			)
+		)

Commit message: 改番
Other:
- board text added: "7 segments LED with HC595 v0.2"
- board text removed: "7 segments LED with HC595 v0.1"
Changed lines of the file:
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@@
 		)
 	)
-	(gr_text "7 segments LED with HC595 v0.1"
+	(gr_text "7 segments LED with HC595 v0.2"
 		(at 125.73 139.7 0)
 		(layer "F.SilkS")
