File: boards/addons/01_basic_digital_io/01_basic_digital_io.kicad_sch (KiCad schematic)
At the start: 1 part, among them J1 Conn_02x15_Odd_Even

Commit message: 作り直した
Parts:
- added D1, D2: LED, LED_THT:LED_D5.0mm, symbol Device:LED
- added R1, R2, R3, R4: R, Resistor_THT:R_Axial_DIN0207_L6.3mm_D2.5mm_P10.16mm_Horizontal, symbol Device:R
- added SW1, SW2: SW_Push, Button_Switch_THT:SW_PUSH-12mm, symbol Switch:SW_Push
Connections:
- net +3.3V: now also R1.1, R2.1
- net GND: now also D1.1 (K), D2.1 (K), SW1.2, SW2.2
- net GP0: now also R1.2, SW1.1
- net GP1: now also R2.2, SW2.1
- net GP2: now also R3.1
- net GP3: now also R4.1
- net SPI_MISO: no longer J1.6 (Pin_6)
- new net: D1.2 (A), R3.2
- new net: D2.2 (A), R4.2
- new net SPI_MOSI: J1.6 (Pin_6)
