File: boards/addons/01_basic_digital_io/01_basic_digital_io.kicad_pcb (KiCad board)
At the start: 2 copper layers, 47 x 72 mm, 1 part, among them J1 Conn_02x15_Odd_Even

Commit message: 作り直した
Parts:
- added D1: LED, LED_THT:LED_D5.0mm, F.Cu at (142.2, 99.1)
- added D2: LED, LED_THT:LED_D5.0mm, F.Cu at (162.6, 99.1)
- added R1: R, Resistor_THT:R_Axial_DIN0207_L6.3mm_D2.5mm_P10.16mm_Horizontal, F.Cu at (147.3, 82.5)
- added R2: R, Resistor_THT:R_Axial_DIN0207_L6.3mm_D2.5mm_P10.16mm_Horizontal, F.Cu at (167.6, 82.5)
- added R3: R, Resistor_THT:R_Axial_DIN0207_L6.3mm_D2.5mm_P10.16mm_Horizontal, F.Cu at (137.2, 78.7)
- added R4: R, Resistor_THT:R_Axial_DIN0207_L6.3mm_D2.5mm_P10.16mm_Horizontal, F.Cu at (157.5, 78.7)
- added SW1: SW_Push, Button_Switch_THT:SW_PUSH-12mm, F.Cu at (136.0, 114.3)
- added SW2: SW_Push, Button_Switch_THT:SW_PUSH-12mm, F.Cu at (156.3, 114.3)
Routing:
- net /GP1: track 0.00 -> 62.0 mm
- net /GP0: track 0.00 -> 48.2 mm
- net +3.3V: track 0.00 -> 31.2 mm
- net /GP2: track 0.00 -> 18.0 mm
- net /GP3: track 0.00 -> 16.2 mm
- net Net-(D2-A): track 0.00 -> 9.72 mm
- net Net-(D1-A): track 0.00 -> 9.72 mm
- added copper zone on B.Cu, net GND
Other:
- board text added: "Basic Digital IO Board for trainer"

Commit message: 配線いじり
Routing:
- net /GP1: track 62.0 -> 73.8 mm
- net /GP0: track 48.2 -> 60.0 mm
Changed lines of the file:
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@@
+	)
+	(segment
+		(start 167.64 113.17)
+		(end 157.48 113.17)
+		(width 0.3)
+		(layer "F.Cu")
+		(net 2)
+	)
+	(segment
+		(start 157.48 113.17)
+		(end 156.31 114.34)
+		(width 0.3)
+		(layer "F.Cu")
+		(net 2)
 	)
 	(segment
@@
 		(width 0.3)
 		(layer "F.Cu")
+		(net 6)
+	)
+	(segment
+		(start 147.32 113.17)
+		(end 137.16 113.17)
+		(width 0.3)
+		(layer "F.Cu")
+		(net 6)
+	)
+	(segment
+		(start 137.16 113.17)
+		(end 135.99 114.34)
+		(width 0.3)
+		(layer "F.Cu")
