File: boards/addons/00_template/00_template.kicad_sch (KiCad schematic)
At the start: 1 part, among them J1 Conn_02x15_Odd_Even

Commit message: ミス修正
Connections:
- net SPI_MISO: no longer J1.6 (Pin_6)
- new net SPI_MOSI: J1.6 (Pin_6)
Changed lines of the file:
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@@
 		)
 	)
-	(label "SPI_MISO"
+	(label "SPI_MOSI"
 		(at 27.94 64.77 0)
 		(effects

Commit message: テンプレミスの修正
Connections:
- net SPI_CS: now also J1.7 (Pin_7); no longer J1.8 (Pin_8)
- net SPI_MISO: now also J1.8 (Pin_8); no longer J1.7 (Pin_7)
- net GP8 renamed GP6
Changed lines of the file:
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@@
 	(label "AD2"
 		(at 27.94 82.55 0)
+		(fields_autoplaced yes)
 		(effects
 			(font
@@
 	(label "SPI_SCK"
 		(at 27.94 36.83 0)
+		(fields_autoplaced yes)
 		(effects
 			(font
@@
 		)
 	)
-	(label "GP8"
+	(label "GP6"
 		(at 27.94 77.47 0)
+		(fields_autoplaced yes)
 		(effects
 			(font
@@
 	(label "I2C_SCL"
 		(at 27.94 41.91 0)
+		(fields_autoplaced yes)
 		(effects
 			(font
@@
 	(label "GP1"
 		(at 27.94 31.75 0)
+		(fields_autoplaced yes)
 		(effects
 			(font
@@
 	(label "GP7"
 		(at 27.94 24.13 0)
+		(fields_autoplaced yes)
 		(effects
 			(font
@@
 	(label "UART_PICO_TX"
 		(at 27.94 59.69 0)
+		(fields_autoplaced yes)
 		(effects
 			(font
@@
 	(label "GP5"
 		(at 27.94 26.67 0)
+		(fields_autoplaced yes)
 		(effects
 			(font
@@
 	(label "GP3"
 		(at 27.94 29.21 0)
+		(fields_autoplaced yes)
 		(effects
 			(font
@@
 	(label "AD1"
 		(at 27.94 21.59 0)
+		(fields_autoplaced yes)
 		(effects
 			(font
@@
 	(label "AD3"
 		(at 27.94 19.05 0)
+		(fields_autoplaced yes)
 		(effects
 			(font
@@
 	(label "UART_PICO_RX"
 		(at 27.94 62.23 0)
+		(fields_autoplaced yes)
 		(effects
 			(font
@@
 	(label "GP4"
 		(at 27.94 74.93 0)
+		(fields_autoplaced yes)
 		(effects
 			(font
@@
 	(label "GP2"
 		(at 27.94 72.39 0)
+		(fields_autoplaced yes)
 		(effects
 			(font
@@
 	)
 	(label "SPI_CS"
-		(at 27.94 67.31 0)
+		(at 27.94 34.29 0)
+		(fields_autoplaced yes)
 		(effects
 			(font
@@
 	(label "I2C_SDA"
 		(at 27.94 39.37 0)
+		(fields_autoplaced yes)
 		(effects
 			(font
@@
 	(label "GP0"
 		(at 27.94 69.85 0)
+		(fields_autoplaced yes)
 		(effects
 			(font
@@
 	(label "SPI_MOSI"
 		(at 27.94 64.77 0)
+		(fields_autoplaced yes)
 		(effects
 			(font
@@
 	)
 	(label "SPI_MISO"
-		(at 27.94 34.29 0)
+		(at 27.94 67.31 0)
+		(fields_autoplaced yes)
 		(effects
 			(font
@@
 	(label "AD0"
 		(at 27.94 80.01 0)
+		(fields_autoplaced yes)
 		(effects
 			(font
