File: boards/addons/02_7seg_direct/02_7seg_direct.kicad_pcb (KiCad board)
At the start: 2 copper layers, 47 x 72 mm, 12 parts, among them J1 Conn_02x15_Odd_Even, U2 74AHC541

Commit message: 配線いじり
Routing:
- net Net-(U1-C): track 36.3 -> 40.0 mm
- net Net-(U1-E): track 21.5 -> 25.2 mm
- net Net-(U1-D): track 27.7 -> 31.3 mm
- net Net-(U1-DP): track 24.0 -> 27.0 mm
- net Net-(U1-B): track 39.2 -> 40.6 mm
- net Net-(U1-A): track 40.9 -> 41.6 mm
- net Net-(U1-G): track 14.3 -> 14.9 mm
Changed lines of the file:
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@@
 	)
 	(segment
-		(start 158.496 115.316)
+		(start 153.416 115.316)
 		(end 168.656 115.316)
 		(width 0.2)
@@
 	)
 	(segment
+		(start 151.13 113.03)
+		(end 153.416 115.316)
+		(width 0.2)
+		(layer "F.Cu")
+		(net 34)
+	)
+	(segment
 		(start 151.13 106.68)
-		(end 151.13 107.95)
-		(width 0.2)
-		(layer "F.Cu")
-		(net 34)
-	)
-	(segment
-		(start 151.13 107.95)
-		(end 158.496 115.316)
+		(end 151.13 113.03)
 		(width 0.2)
 		(layer "F.Cu")
@@
 	)
 	(segment
-		(start 158.75 102.87)
-		(end 151.13 102.87)
-		(width 0.2)
-		(layer "F.Cu")
-		(net 35)
-	)
-	(segment
-		(start 148.59 105.41)
-		(end 148.59 106.68)
-		(width 0.2)
-		(layer "F.Cu")
-		(net 35)
-	)
-	(segment
-		(start 151.13 102.87)
-		(end 148.59 105.41)
-		(width 0.2)
-		(layer "F.Cu")
-		(net 35)
-	)
-	(segment
 		(start 160.02 101.6)
 		(end 158.75 102.87)
@@
 	)
 	(segment
+		(start 150.114 102.87)
+		(end 148.59 104.394)
+		(width 0.2)
+		(layer "F.Cu")
+		(net 35)
+	)
+	(segment
+		(start 148.59 104.394)
+		(end 148.59 106.68)
+		(width 0.2)
+		(layer "F.Cu")
+		(net 35)
+	)
+	(segment
+		(start 158.75 102.87)
+		(end 150.114 102.87)
+		(width 0.2)
+		(layer "F.Cu")
+		(net 35)
+	)
+	(segment
+		(start 146.05 107.696)
+		(end 146.05 106.68)
+		(width 0.2)
+		(layer "F.Cu")
+		(net 36)
+	)
+	(segment
+		(start 160.02 104.14)
+		(end 151.13 104.14)
+		(width 0.2)
+		(layer "F.Cu")
+		(net 36)
+	)
+	(segment
+		(start 149.86 107.696)
+		(end 149.098 108.458)
+		(width 0.2)
+		(layer "F.Cu")
+		(net 36)
+	)
+	(segment
 		(start 151.13 104.14)
 		(end 149.86 105.41)
@@
 	)
 	(segment
+		(start 146.558 106.68)
+		(end 146.05 106.68)
+		(width 0.2)
+		(layer "F.Cu")
+		(net 36)
+	)
+	(segment
+		(start 146.812 108.458)
+		(end 146.05 107.696)
+		(width 0.2)
+		(layer "F.Cu")
+		(net 36)
+	)
+	(segment
 		(start 149.86 105.41)
 		(end 149.86 107.696)
@@
 	)
 	(segment
-		(start 146.558 106.68)
-		(end 146.05 106.68)
-		(width 0.2)
-		(layer "F.Cu")
-		(net 36)
-	)
-	(segment
 		(start 162.56 101.6)
 		(end 160.02 104.14)
@@
 	)
 	(segment
-		(start 149.86 107.696)
-		(end 149.098 108.458)
-		(width 0.2)
-		(layer "F.Cu")
-		(net 36)
-	)
-	(segment
-		(start 160.02 104.14)
-		(end 151.13 104.14)
-		(width 0.2)
-		(layer "F.Cu")
-		(net 36)
-	)
-	(segment
-		(start 146.812 108.458)
-		(end 146.05 107.696)
-		(width 0.2)
-		(layer "F.Cu")
-		(net 36)
-	)
-	(segment
-		(start 146.05 107.696)
-		(end 146.05 106.68)
-		(width 0.2)
-		(layer "F.Cu")
-		(net 36)
-	)
-	(segment
 		(start 160.02 116.84)
-		(end 152.4 116.84)
+		(end 146.05 116.84)
 		(width 0.2)
 		(layer "F.Cu")
@@
 	)
 	(segment
-		(start 152.4 116.84)
-		(end 143.51 107.95)
+		(start 146.05 116.84)
+		(end 143.51 114.3)
 		(width 0.2)
 		(layer "F.Cu")
@@
 	)
 	(segment
-		(start 143.51 107.95)
+		(start 143.51 114.3)
 		(end 143.51 106.68)
 		(width 0.2)
@@
 	(segment
 		(start 140.97 106.68)
-		(end 140.97 108.077)
-		(width 0.2)
-		(layer "F.Cu")
-		(net 38)
-	)
-	(segment
-		(start 151.003 118.11)
-		(end 161.29 118.11)
-		(width 0.2)
-		(layer "F.Cu")
-		(net 38)
-	)
-	(segment
-		(start 140.97 108.077)
-		(end 151.003 118.11)
+		(end 140.97 114.3)
 		(width 0.2)
 		(layer "F.Cu")
@@
 	)
 	(segment
-		(start 138.43 107.95)
-		(end 149.86 119.38)
-		(width 0.2)
-		(layer "F.Cu")
-		(net 39)
-	)
-	(segment
-		(start 149.86 119.38)
-		(end 165.1 119.38)
-		(width 0.2)
-		(layer "F.Cu")
-		(net 39)
+		(start 144.78 118.11)
+		(end 161.29 118.11)
+		(width 0.2)
+		(layer "F.Cu")
+		(net 38)
+	)
+	(segment
+		(start 140.97 114.3)
+		(end 144.78 118.11)
+		(width 0.2)
+		(layer "F.Cu")
+		(net 38)
 	)
 	(segment
 		(start 138.43 106.68)
-		(end 138.43 107.95)
+		(end 138.43 114.3)
 		(width 0.2)
 		(layer "F.Cu")
@@
 	)
 	(segment
+		(start 143.51 119.38)
+		(end 165.1 119.38)
+		(width 0.2)
+		(layer "F.Cu")
+		(net 39)
+	)
+	(segment
+		(start 138.43 114.3)
+		(end 143.51 119.38)
+		(width 0.2)
+		(layer "F.Cu")
+		(net 39)
+	)
+	(segment
 		(start 167.64 99.06)
-		(end 142.24 99.06)
-		(width 0.2)
-		(layer "F.Cu")
-		(net 40)
-	)
-	(segment
-		(start 142.24 99.06)
-		(end 135.89 105.41)
-		(width 0.2)
-		(layer "F.Cu")
-		(net 40)
-	)
-	(segment
-		(start 135.89 105.41)
+		(end 139.954 99.06)
+		(width 0.2)
+		(layer "F.Cu")
+		(net 40)
+	)
+	(segment
+		(start 135.89 103.124)
 		(end 135.89 106.68)
 		(width 0.2)
@@
 	)
 	(segment
+		(start 139.954 99.06)
+		(end 135.89 103.124)
+		(width 0.2)
+		(layer "F.Cu")
+		(net 40)
+	)
+	(segment
+		(start 167.64 101.6)
+		(end 166.37 100.33)
+		(width 0.2)
+		(layer "F.Cu")
+		(net 41)
+	)
+	(segment
+		(start 134.112 108.458)
+		(end 133.35 107.696)
+		(width 0.2)
+		(layer "F.Cu")
+		(net 41)
+	)
+	(segment
 		(start 166.37 100.33)
-		(end 142.24 100.33)
+		(end 140.97 100.33)
+		(width 0.2)
+		(layer "F.Cu")
+		(net 41)
+	)
+	(segment
+		(start 136.398 108.458)
+		(end 134.112 108.458)
+		(width 0.2)
+		(layer "F.Cu")
+		(net 41)
+	)
+	(segment
+		(start 137.16 107.696)
+		(end 136.398 108.458)
 		(width 0.2)
 		(layer "F.Cu")
@@
 	)
 	(segment
-		(start 136.398 108.458)
-		(end 134.112 108.458)
-		(width 0.2)
-		(layer "F.Cu")
-		(net 41)
-	)
-	(segment
-		(start 137.16 105.41)
+		(start 137.16 104.14)
 		(end 137.16 107.696)
 		(width 0.2)
@@
 	)
 	(segment
-		(start 142.24 100.33)
-		(end 137.16 105.41)
-		(width 0.2)
-		(layer "F.Cu")
-		(net 41)
-	)
-	(segment
-		(start 167.64 101.6)
-		(end 166.37 100.33)
-		(width 0.2)
-		(layer "F.Cu")
-		(net 41)
-	)
-	(segment
-		(start 134.112 108.458)
-		(end 133.35 107.696)
-		(width 0.2)
-		(layer "F.Cu")
-		(net 41)
-	)
-	(segment
-		(start 137.16 107.696)
-		(end 136.398 108.458)
-		(width 0.2)
-		(layer "F.Cu")
+		(start 140.97 100.33)
+		(end 137.16 104.14)
+		(width 0.2)
+		(layer "F.Cu")
