File: boards/addons/05_analog_input/05_analog_input.kicad_sch (KiCad schematic)
At the start: 3 parts, among them J1 Conn_02x15_Odd_Even

Commit message: CdS の回路とコンデンサを追加
Parts:
- added C1: 10uF, Capacitor_THT:CP_Radial_D5.0mm_P2.00mm, symbol Device:C
- added C2: 0.1uF, Capacitor_THT:C_Disc_D5.1mm_W3.2mm_P5.00mm, symbol Device:C
- added R1: R, Resistor_THT:R_Radial_Power_L11.0mm_W7.0mm_P5.00mm, symbol Device:R
- added R2: R, Resistor_THT:R_Axial_DIN0207_L6.3mm_D2.5mm_P10.16mm_Horizontal, symbol Device:R
Connections:
- net +3.3V: now also C1.1, C2.1, R1.1
- net AD2: now also R1.2, R2.1
- net GND: now also C1.2, C2.2, R2.2
